File: PCB/Adm3aXep80/Adm3aXep80.kicad_sch (KiCad schematic)
At the start: 10 parts, among them J1 Conn_Coaxial, J2 Conn_01x09, J22 Conn_01x13, J8 Conn_01x13

Commit message: PCB
Parts:
- removed A1: RaspberryPi_Pico, Module:RaspberryPi_Pico_Common_Unspecified, symbol MCU_Module:RaspberryPi_Pico
- removed J1: Conn_Coaxial, Atari:CUI_RCJ-043, symbol Connector:Conn_Coaxial
- removed U1: ~, Package_DIP:DIP-12_W7.62mm_LongPads, symbol xep80:Level_Shifter
- added D1, D2: 1N4148, Diode_THT:D_DO-35_SOD27_P7.62mm_Horizontal, symbol Diode:1N4148
- added D3, D4: LED, LED_THT:LED_D3.0mm, symbol Device:LED
- added H1, H2, H3, H4: MountingHole, MountingHole:MountingHole_3.2mm_M3, symbol Mechanical:MountingHole
- added J1: HDMI, Package_DIP:DIP-40_W25.4mm_Socket_LongPads, symbol Connector_Generic:Conn_02x20_Counter_Clockwise
- added J3: Conn_Coaxial, RCA:RCA-Phono_CUI-Devices_RCJ-01X_Horizontal, symbol Connector:Conn_Coaxial
- added J4: prog, Connector_PinHeader_2.54mm:PinHeader_1x01_P2.54mm_Vertical, symbol Connector_Generic:Conn_01x01
- added J5: Conn_01x04, Button_Switch_THT:SW_Tactile_SKHH_Angled, symbol Connector_Generic:Conn_01x04
- added R1, R5, R6, R7: 1K, Resistor_THT:R_Axial_DIN0207_L6.3mm_D2.5mm_P10.16mm_Horizontal, symbol Device:R_Small
- added U1: 74125, Package_DIP:DIP-14_W7.62mm_Socket, symbol 74xx_IEEE:74125
- R2: value 1K -> 2.2K
Connections:
- net +3V3: now also D3.2 (A), D4.2 (A), U1.14 (VCC), U1.14 (VCC), U1.14 (VCC), U1.14 (VCC)
- net CLK_N: now also J1.30 (Pin_30)
- net CLK_P: now also J1.29 (Pin_29)
- net DVI_D0N: now also J1.27 (Pin_27)
- net DVI_D0P: now also J1.26 (Pin_26)
- net DVI_D1N: now also J1.25 (Pin_25)
- net DVI_D1P: now also J1.24 (Pin_24)
- net DVI_D2N: now also J1.22 (Pin_22)
- net DVI_D2P: now also J1.21 (Pin_21)
- net GND: now also J1.23 (Pin_23), J1.28 (Pin_28), J1.33 (Pin_33), J1.38 (Pin_38), J3.2 (Ext), J5.1 (Pin_1), R5.1, U1.7 (GND), U1.7 (GND), U1.7 (GND), U1.7 (GND)
- net JOY1: now also U1.12 (D)
- net JOY2: now also U1.6 (O)
- net SERIN: now also A2.4 (GPIO2), R6.2, U1.11 (O), U1.8 (O); no longer A2.5 (GPIO3)
- net SEROUT: now also A2.5 (GPIO3), R7.2, U1.2 (D), U1.5 (D); no longer A2.6 (GPIO4)
- net SIORDY: now also D1.2 (A); no longer A2.39 (VSYS), J2.7 (Pin_7)
- net SIO_Motor: now also R5.2, U1.9 (D); no longer R2.2
- net SIO_Proceed: now also U1.3 (O)
- net JOYEN\: now reaches A2.7 (GPIO5)
- net JOYEN\: now also U1.13 (EN), U1.4 (EN)
- net at R3.1, R4.1: now also J3.1 (In)
- new net: A2.39 (VSYS), D1.1 (K), D2.1 (K)
- new net: D4.1 (K), R7.1
- new net: D3.1 (K), R6.1
- new net: J4.1 (Pin_1), J5.2 (Pin_2)
- new net JOY5V: D2.2 (A), J2.7 (Pin_7), R1.2
- new net JOYEN: A2.6 (GPIO4), R1.1, R2.2, U1.1 (EN), U1.10 (EN)
Other:
- moved on the sheet: A2, R3, R4
